File: KiCad/Core 2x2/Core 2x2/Core 2x2.kicad_pcb (KiCad board)
At the start: 2 copper layers, 138 parts, among them J1 Conn_01x02_Female, J10 Conn_02x03_Odd_Even, J11 02x10, J12 Conn_01x09_Male, J13 Conn_01x03_Male, J2 Conn_02x03_Odd_Even, J3 02x10, J4 Conn_02x03_Odd_Even, J5 02x10, J6 Conn_02x03_Odd_Even, J7 Conn_02x03_Odd_Even, J8 Conn_02x03_Odd_Even, J9 02x10, Q1 2STF2550, U1 SN74AHC125, U2 SN74AHC125, U3 LT8608, U4 LT8608, U5 SN74AHC125, U6 SN74AHC125, U7 ADAU1452, U8 M95M01, Y1 12.288MHz

Commit message: Progress Commit
Parts:
- added C49: 100n, Capacitor_SMD:C_0402_1005Metric, F.Cu at (42.0, 64.0)
- added C50: 100n, Capacitor_SMD:C_0402_1005Metric, F.Cu at (181.5, 64.0)
- added C51: 100n, Capacitor_SMD:C_0402_1005Metric, F.Cu at (209.5, 64.0)
- added C52: 100n, Capacitor_SMD:C_0402_1005Metric, F.Cu at (237.5, 64.0)
- added J14: Conn_02x03_Odd_Even, Connector_PinHeader_2.54mm:PinHeader_2x03_P2.54mm_Vertical_SMD, F.Cu at (28.0, 70.0)
- added J15: 02x10, Connector_PinHeader_2.54mm:PinHeader_2x10_P2.54mm_Horizontal, F.Cu at (20.5, 61.0)
- added J16: Conn_02x03_Odd_Even, Connector_PinHeader_2.54mm:PinHeader_2x03_P2.54mm_Vertical_SMD, F.Cu at (167.5, 70.0)
- added J17: 02x10, Connector_PinHeader_2.54mm:PinHeader_2x10_P2.54mm_Horizontal, F.Cu at (160.0, 61.0)
- added J18: Conn_02x03_Odd_Even, Connector_PinHeader_2.54mm:PinHeader_2x03_P2.54mm_Vertical_SMD, F.Cu at (195.5, 70.0)
- added J19: 02x10, Connector_PinHeader_2.54mm:PinHeader_2x10_P2.54mm_Horizontal, F.Cu at (188.0, 61.0)
- added J20: Conn_02x03_Odd_Even, Connector_PinHeader_2.54mm:PinHeader_2x03_P2.54mm_Vertical_SMD, F.Cu at (223.5, 70.0)
- added J21: 02x10, Connector_PinHeader_2.54mm:PinHeader_2x10_P2.54mm_Horizontal, F.Cu at (216.0, 61.0)
- added R63: 33R, Resistor_SMD:R_0402_1005Metric, F.Cu at (67.0, 64.0)
- added R64: 33R, Resistor_SMD:R_0402_1005Metric, F.Cu at (69.0, 64.0)
- added R65: 33R, Resistor_SMD:R_0402_1005Metric, F.Cu at (39.0, 64.0)
- added R66: 33R, Resistor_SMD:R_0402_1005Metric, F.Cu at (41.0, 64.0)
- added R67: 33R, Resistor_SMD:R_0402_1005Metric, F.Cu at (178.5, 64.0)
- added R68: 33R, Resistor_SMD:R_0402_1005Metric, F.Cu at (180.5, 64.0)
- added R69: 33R, Resistor_SMD:R_0402_1005Metric, F.Cu at (206.5, 64.0)
- added R70: 33R, Resistor_SMD:R_0402_1005Metric, F.Cu at (208.5, 64.0)
- added R71: 33R, Resistor_SMD:R_0402_1005Metric, F.Cu at (234.5, 64.0)
- added R72: 33R, Resistor_SMD:R_0402_1005Metric, F.Cu at (236.5, 64.0)
- added R73: 33R, Resistor_SMD:R_0402_1005Metric, F.Cu at (177.5, 64.0)
- added R74: 33R, Resistor_SMD:R_0402_1005Metric, F.Cu at (179.5, 64.0)
- added R75: 33R, Resistor_SMD:R_0402_1005Metric, F.Cu at (205.5, 64.0)
- added R76: 33R, Resistor_SMD:R_0402_1005Metric, F.Cu at (207.5, 64.0)
- added R77: 33R, Resistor_SMD:R_0402_1005Metric, F.Cu at (233.5, 64.0)
- added R78: 33R, Resistor_SMD:R_0402_1005Metric, F.Cu at (235.5, 64.0)
- added REF**: PCB_Board_70x43, Library:PCB_Board_70x43, Cmts.User at (59.8, 7.25)
- added REF**: PCB_Board_70x43, Library:PCB_Board_70x43, Cmts.User at (203.8, 7.25)
- added REF**: PCB_Board_70x43, Library:PCB_Board_70x43, Cmts.User at (153.0, 7.50)
- added REF**: PCB_Board_70x43, Library:PCB_Board_70x43, Cmts.User at (108.0, 7.25)
- added U10: SN74AHC125, Package_SO:SOIC-14_3.9x8.7mm_P1.27mm, F.Cu at (179.0, 70.0)
- added U11: SN74AHC125, Package_SO:SOIC-14_3.9x8.7mm_P1.27mm, F.Cu at (207.0, 70.0)
- added U12: SN74AHC125, Package_SO:SOIC-14_3.9x8.7mm_P1.27mm, F.Cu at (235.0, 70.0)
- added U9: SN74AHC125, Package_SO:SOIC-14_3.9x8.7mm_P1.27mm, F.Cu at (39.5, 70.0)
- moved R24 146.6 mm to (34.5, 68.8), turned to 180 degrees
- moved R23 116.6 mm to (62.5, 68.8), turned to 180 degrees
- moved U6 112.0 mm to (67.5, 70.0)
- moved J10 112.0 mm to (56.0, 70.0)
- moved C15 112.0 mm to (70.0, 64.0)
- moved J11 111.5 mm to (48.5, 61.0)
- moved R27 83.0 mm to (95.0, 64.0)
- moved R28 83.0 mm to (97.0, 64.0)
- moved R9 55.5 mm to (40.0, 64.0)
- moved J12 54.1 mm to (184.5, 149.0)
- moved J13 54.1 mm to (184.5, 158.0)
- moved J6 49.9 mm to (167.5, 144.5)
- moved FB1 47.1 mm to (122.0, 93.0), turned to 90 degrees
- moved J7 35.2 mm to (166.5, 156.0)
- moved R4 28.5 mm to (68.0, 64.0)
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Connections:
- C17 pad 1: +3V3 -> /DSP/AVDD
- C18 pad 1: +3V3 -> /DSP/AVDD
- C19 pad 1: +3V3 -> /DSP/AVDD
- C21 pad 1: +3V3 -> /DSP/AVDD
- C23 pad 1: /DSP/IOVDD -> +3V3
- C25 pad 2: VDDA -> /DSP/AVDD
- C29 pad 1: /DSP/IOVDD -> +3V3
- C30 pad 2: VDDA -> /DSP/AVDD
- C32 pad 1: /DSP/IOVDD -> +3V3
- C34 pad 1: /DSP/IOVDD -> +3V3
- C35 pad 1: /DSP/IOVDD -> +3V3
- FB1 pad 1: /DSP/IOVDD -> /DSP/AVDD
- J11 pad 10: /SPI_SS4 -> /SPI_SS3
- J3 pad 13: /SDI0 -> Net-(J3-Pad13)
- J3 pad 7: Net-(J3-Pad7) -> Net-(J2-Pad3)
- J5 pad 10: /SPI_SS4 -> /SPI_SS3
- J5 pad 13: /SDI1 -> Net-(J5-Pad13)
- J5 pad 7: Net-(J5-Pad7) -> Net-(J4-Pad3)
- Q1 pad 3: /DSP/IOVDD -> +3V3
- R1 pad 1: /DSP/SDI0 -> Net-(R1-Pad1)
- R1 pad 2: Net-(R1-Pad2) -> /SDI0
- R10 pad 1: Net-(J5-Pad19) -> Net-(R10-Pad1)
- R10 pad 2: Net-(R10-Pad2) -> /SDI1
- R23 pad 1: Net-(J11-Pad15) -> Net-(R23-Pad1)
- R23 pad 2: Net-(R23-Pad2) -> /SDI2
- R24 pad 1: Net-(J11-Pad19) -> Net-(R24-Pad1)
- R24 pad 2: Net-(R24-Pad2) -> /SDI3
- R27 pad 1: Net-(J11-Pad13) -> Net-(J5-Pad15)
- R28 pad 1: Net-(J11-Pad17) -> Net-(J5-Pad19)
- R3 pad 1: /DSP/SDI1 -> Net-(J5-Pad17)
- R31 pad 2: /DSP/SDI0 -> /SDI0
- R34 pad 2: /DSP/SDI1 -> /SDI1
- R35 pad 2: /DSP/LRCLKI2 -> /DSP/BCLKI2
- R36 pad 2: /DSP/BCLKI2 -> /DSP/LRCLKI2
- R37 pad 2: /DSP/SDI2 -> /SDI2
- R38 pad 2: /DSP/LRCLKI3 -> /DSP/BCLKI3
- R39 pad 2: /DSP/BCLKI3 -> /DSP/LRCLKI3
- R4 pad 1: Net-(J5-Pad17) -> Net-(J11-Pad17)
- R40 pad 2: /DSP/SDI3 -> /SDI3
- R49 pad 2: /DSP/IOVDD -> +3V3
- R9 pad 1: Net-(J5-Pad15) -> Net-(J15-Pad17)
- U1 pad 2: /SDI0 -> Net-(J3-Pad13)
- U1 pad 3: Net-(R1-Pad2) -> Net-(R1-Pad1)
- U2 pad 10: Net-(R4-Pad2) -> Net-(R3-Pad2)
- U2 pad 13: Net-(R10-Pad2) -> Net-(R28-Pad2)
- U2 pad 2: /SDI1 -> Net-(J5-Pad13)
- U2 pad 3: Net-(R3-Pad2) -> Net-(R10-Pad1)
- U2 pad 6: Net-(R9-Pad2) -> Net-(R27-Pad2)
- U6 pad 10: Net-(R28-Pad2) -> Net-(R4-Pad2)
- U6 pad 13: Net-(R24-Pad2) -> Net-(R64-Pad2)
- U6 pad 2: /DSP/SDO2 -> Net-(J11-Pad13)
- U6 pad 3: Net-(R27-Pad2) -> Net-(R23-Pad1)
- U6 pad 5: /DSP/BCLKO2 -> /DSP/BCLKI2
- U6 pad 6: Net-(R23-Pad2) -> Net-(R63-Pad2)
- U6 pad 9: /DSP/LRCLKO2 -> /DSP/LRCLKI2
- U7 pad 15: +3V3 -> /DSP/AVDD
- U7 pad 18: /DSP/IOVDD -> +3V3
- U7 pad 2: /DSP/IOVDD -> +3V3
- U7 pad 38: /DSP/IOVDD -> +3V3
- U7 pad 56: /DSP/IOVDD -> +3V3
- U7 pad 7: +3V3 -> /DSP/AVDD
Routing:
- net (no net): track 130.0 -> 0.00 mm, vias 1 -> 0
- net /DSP/SDO0: track 0.00 -> 102.8 mm
- net /DSP/LRCLKO0: track 0.00 -> 101.8 mm
- net /DSP/BCLKO0: track 0.00 -> 99.9 mm
- net /SDI3: track 0.00 -> 96.9 mm
- net /DSP/BCLKI3: track 0.00 -> 94.6 mm
- net /DSP/LRCLKI3: track 0.00 -> 88.7 mm, vias 0 -> 2
- net /DSP/SDO1: track 0.00 -> 73.8 mm
- net /DSP/LRCLKO1: track 0.00 -> 72.6 mm
- net /DSP/BCLKO1: track 0.00 -> 70.7 mm
- net /SDI2: track 0.00 -> 67.2 mm
- net /DSP/BCLKI2: track 0.00 -> 65.0 mm
- net /DSP/LRCLKI2: track 0.00 -> 58.6 mm, vias 0 -> 2
- net /DSP/SDO2: track 0.00 -> 48.3 mm
- net /DSP/LRCLKO2: track 0.00 -> 44.9 mm
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Other:
- board outline added: 221.5 x 70.5 mm
- copper layers 2 -> 4
- net class Default: via_dia 0.8 -> 0.6; via_drill 0.4 -> 0.3
