File: KiCad/Core 2x2/Core 2x2/Core 2x2.sch (KiCad schematic (older format))
At the start: 67 parts, among them J1 Conn_01x02_Female, J10 Conn_02x03_Odd_Even, J11 02x10, J12 Conn_01x09_Male, J13 Conn_01x03_Male, J2 Conn_02x03_Odd_Even, J3 02x10, J4 Conn_02x03_Odd_Even, J5 02x10, J6 Conn_02x03_Odd_Even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

Commit message: Progress Commit
Parts:
- removed U2, U6: SN74AHC125, Package_SO:SOIC-14_3.9x8.7mm_P1.27mm, symbol FA-Library:SN74AHC125
- added C49, C50, C51, C52: 100n, Capacitor_SMD:C_0402_1005Metric, symbol Device:C_Small
- added J14, J16, J18, J20: Conn_02x03_Odd_Even, Connector_PinHeader_2.54mm:PinHeader_2x03_P2.54mm_Vertical_SMD, symbol Connector_Generic:Conn_02x03_Odd_Even
- added J15, J17, J19, J21: 02x10, Connector_PinHeader_2.54mm:PinHeader_2x10_P2.54mm_Horizontal, symbol Connector_Generic:Conn_02x10_Odd_Even
- added R63, R64, R65, R66, R67, R68, R69, R70, R71, R72, R73, R74, R75, R76, R77, R78: 33R, Resistor_SMD:R_0402_1005Metric, symbol Device:R_Small
- added U10, U11, U12, U2, U6, U9: SN74AHC125, Package_SO:SOIC-14_3.9x8.7mm_P1.27mm, symbol Core-2x2-rescue:SN74AHC125-FA-Library
- U1, U5: symbol FA-Library:SN74AHC125 -> Core-2x2-rescue:SN74AHC125-FA-Library
- U3, U4: symbol FA-Library:LT8606 -> Core-2x2-rescue:LT8606-FA-Library
Connections:
- net labels added: SDI2, SDI3
- wire segments 407 -> 705
Other:
- note added: "SDA\nBCLK\nLRCLK\nMCLK"
- moved on the sheet: C1, C10, C11, C12, C13, C14, C16, C2, C3, C5, C6, C7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
