File: KiCad/Core 1x1/Core 1x1.kicad_pcb (KiCad board)
At the start: 4 copper layers, 90 x 55 mm, 171 parts, among them J100 Conn_01x02_Female, J101 02x10, J102 02x10, J103 Conn_02x05_Odd_Even, J12 Conn_01x09_Male, J13 Conn_01x03_Male, Q1 2STF2550, U3 LT8608, U4 LT8608, U7 ADAU1452, U8 M95M01, Y1 12.288MHz

Commit message: Pre-release commit
Parts:
- removed the C1 at (40.5, 15.3)
- removed the C10 at (34.5, -8.00)
- removed the C11 at (34.5, 0.00)
- removed the C13 at (34.5, -3.00)
- removed the C14 at (40.5, -6.00)
- removed the C2 at (34.5, 9.50)
- removed C28, C31: 100p, Capacitor_SMD:C_0402_1005Metric
- removed the C3 at (34.5, 17.5)
- removed C37, C40, C43, C46: 100n, Capacitor_SMD:C_0402_1005Metric
- removed C38, C41, C44, C47: 1u, Capacitor_SMD:C_0402_1005Metric
- removed the C7 at (34.5, 14.5)
- removed the C8 at (40.5, 11.5)
- removed the C9 at (40.5, -2.00)
- removed J12: Conn_01x09_Male, Connector_JST:JST_PH_B9B-PH-K_1x09_P2.00mm_Vertical
- removed J13: Conn_01x03_Male, Connector_JST:JST_PH_B3B-PH-K_1x03_P2.00mm_Vertical
- removed JP2, JP3: Jumper_NC_Dual, Connector_PinHeader_2.54mm:PinHeader_1x03_P2.54mm_Vertical
- removed L1, L2: 10u, Inductor_SMD:L_Bourns_SRP7028A_7.3x6.6mm
- removed the R1 at (-18.2, -18.0)
- removed the R11 at (34.5, 10.5)
- removed the R12 at (34.5, 16.5)
- removed the R13 at (34.5, 15.5)
- removed the R14 at (50.0, 6.49)
- removed the R15 at (50.5, -4.50)
- removed the R16 at (38.5, 0.00)
- removed the R2 at (-16.2, -18.0)
- removed the R25 at (28.8, -18.0)
- removed the R26 at (30.8, -18.0)
- removed the R5 at (-17.2, -18.0)
- removed the R7 at (38.5, 17.5)
- removed the R8 at (34.5, 8.50)
- removed REF** (x2): PCB_Board_70x43, Library:PCB_Board_70x43
- removed TP1, TP10, TP11, TP12, TP13, TP14, TP15, TP16, TP17, TP18, TP19, TP2, TP20, TP21, TP22, TP23, TP24, TP3, TP31, TP32, TP33, TP34, TP35, TP36, TP37, TP38, TP39, TP4, TP40, TP41, TP42, TP43, TP44, TP45, TP46, TP47, TP48, TP5, TP6, TP7, TP8, TP9: TestPoint, TestPoint:TestPoint_Pad_D1.0mm
- removed the U3 at (37.5, 13.5)
- added C100: 4.7u, Capacitor_SMD:C_0805_2012Metric, F.Cu at (27.8, 18.2)
- added C101: 4.7u, Capacitor_SMD:C_0805_2012Metric, F.Cu at (27.8, 14.8)
- added C102: 4.7u, Capacitor_SMD:C_0402_1005Metric, F.Cu at (-32.8, 18.2)
- added C103: 100n, Capacitor_SMD:C_0402_1005Metric, F.Cu at (-32.8, 19.2)
- added C106: 10n, Capacitor_SMD:C_0402_1005Metric, F.Cu at (-32.8, 9.25)
- added C107: 1u, Capacitor_SMD:C_0402_1005Metric, F.Cu at (-32.8, 10.2)
- added C15: 100p, Capacitor_SMD:C_0402_1005Metric, F.Cu at (-19.8, 7.50)
- added C17: 100p, Capacitor_SMD:C_0402_1005Metric, F.Cu at (-21.8, 7.50)
- added C200: 10u, Capacitor_SMD:C_0805_2012Metric, F.Cu at (33.2, 14.0)
- added C201: 1u, Capacitor_SMD:C_0402_1005Metric, F.Cu at (43.0, 12.5)
- added C202: 10n, Capacitor_SMD:C_0402_1005Metric, F.Cu at (43.0, 11.5)
- added C203: 10n, Capacitor_SMD:C_0402_1005Metric, F.Cu at (39.5, 5.99)
- added C204: 2.2p, Capacitor_SMD:C_0402_1005Metric, F.Cu at (40.5, 6.00)
- added C205: 120p, Capacitor_SMD:C_0402_1005Metric, F.Cu at (41.0, 4.50)
- added C206: 10p, Capacitor_SMD:C_0402_1005Metric, F.Cu at (34.5, 5.00)
- added C207: 10u, Capacitor_SMD:C_0805_2012Metric, F.Cu at (30.2, 7.00)
- added C208: 10u, Capacitor_SMD:C_0805_2012Metric, F.Cu at (30.2, 5.00)
- added C24: 10n, Capacitor_SMD:C_0402_1005Metric, F.Cu at (-38.2, 8.00)
- added C25: 10n, Capacitor_SMD:C_0402_1005Metric, F.Cu at (-38.2, 13.0)
- added C27: 10n, Capacitor_SMD:C_0402_1005Metric, F.Cu at (-38.2, 18.0)
- added C300: 10u, Capacitor_SMD:C_0805_2012Metric, F.Cu at (33.2, 2.00)
- added C301: 1u, Capacitor_SMD:C_0402_1005Metric, F.Cu at (43.0, 0.50)
- added C302: 10n, Capacitor_SMD:C_0402_1005Metric, F.Cu at (43.0, -0.50)
- added C303: 10n, Capacitor_SMD:C_0402_1005Metric, F.Cu at (39.5, -6.00)
- added C304: 2.2p, Capacitor_SMD:C_0402_1005Metric, F.Cu at (40.5, -6.00)
- added C305: 120p, Capacitor_SMD:C_0402_1005Metric, F.Cu at (41.0, -7.50)
- added C306: 10p, Capacitor_SMD:C_0402_1005Metric, F.Cu at (34.5, -7.00)
- added C307: 10u, Capacitor_SMD:C_0805_2012Metric, F.Cu at (30.2, -5.00)
- added C308: 10u, Capacitor_SMD:C_0805_2012Metric, F.Cu at (30.2, -7.00)
- added C34: 100n, Capacitor_SMD:C_0402_1005Metric, F.Cu at (8.50, 18.0)
- added C35: 100n, Capacitor_SMD:C_0402_1005Metric, F.Cu at (4.50, -16.2)
- added C5: 100n, Capacitor_SMD:C_0402_1005Metric, F.Cu at (-3.50, 9.00)
- added D10: BAS516, Diode_SMD:D_SOD-523, F.Cu at (-2.25, 22.0)
- added D11: BAS516, Diode_SMD:D_SOD-523, F.Cu at (-0.75, 22.0)
- added D200: Yellow, Diode_SMD:D_0603_1608Metric, F.Cu at (38.8, 14.2)
- added D201: Green, Diode_SMD:D_0603_1608Metric, F.Cu at (40.2, 14.2)
- added D300: Yellow, Diode_SMD:D_0603_1608Metric, F.Cu at (38.8, 2.25)
- added D301: Green, Diode_SMD:D_0603_1608Metric, F.Cu at (40.2, 2.25)
- added D4: BAS516, Diode_SMD:D_SOD-523, F.Cu at (3.00, -21.2)
- added D5: BAS516, Diode_SMD:D_SOD-523, F.Cu at (-3.00, -21.2)
- added D6: BAS516, Diode_SMD:D_SOD-523, F.Cu at (-5.75, -20.2)
- added D7: BAS516, Diode_SMD:D_SOD-523, F.Cu at (-5.75, -21.8)
- added D8: BAS516, Diode_SMD:D_SOD-523, F.Cu at (2.25, 22.0)
- added D9: BAS516, Diode_SMD:D_SOD-523, F.Cu at (0.75, 22.0)
- added J1: TC2030, Connector:Tag-Connect_TC2030-IDC-NL_2x03_P1.27mm_Vertical, F.Cu at (-22.5, 19.8)
- added J104: 02x10, Connector_PinHeader_2.54mm:PinHeader_2x10_P2.54mm_Vertical, F.Cu at (-35.0, -11.0)
- added J105: Conn_02x03_Odd_Even, Connector_PinHeader_2.54mm:PinHeader_2x03_P2.54mm_Vertical, F.Cu at (-24.8, -4.50)
- added J106: Conn_02x03_Odd_Even, Connector_PinHeader_2.54mm:PinHeader_2x03_P2.54mm_Vertical, F.Cu at (-24.8, 2.00)
- added J107: Conn_02x03_Odd_Even, Connector_PinHeader_2.54mm:PinHeader_2x03_P2.54mm_Vertical, F.Cu at (19.5, 2.00)
- added J108: Conn_02x03_Odd_Even, Connector_PinHeader_2.54mm:PinHeader_2x03_P2.54mm_Vertical, F.Cu at (19.5, -4.50)
- added J109: 02x10, Connector_PinHeader_2.54mm:PinHeader_2x10_P2.54mm_Vertical, F.Cu at (12.0, -11.0)
- added J110: USB_OTG, Connector_USB:USB_Micro-B_Molex-105017-0001, F.Cu at (-29.5, 24.8)
- added J2: JST_XH_B2B, Connector_JST:JST_XH_B2B-XH-A_1x02_P2.50mm_Vertical, F.Cu at (-39.8, -16.2)
- added J3: JST_XH_B2B, Connector_JST:JST_XH_B2B-XH-A_1x02_P2.50mm_Vertical, F.Cu at (-39.8, -9.50)
- added L100: 4.7u, Farving_Labs_Library:L_Pulse_PA4546.XXXNLT, F.Cu at (24.5, 16.5)
- added L200: 10u, Farving_Labs_Library:L_Pulse_PA4546.XXXNLT, F.Cu at (29.5, 10.5)
- added L300: 10u, Farving_Labs_Library:L_Pulse_PA4546.XXXNLT, F.Cu at (29.5, -1.50)
- added NT1: Net-Tie_2, NetTie:NetTie-2_SMD_Pad0.5mm, B.Cu at (1.25, 5.50)
- added Q2: BC846BS, Package_TO_SOT_SMD:SOT-363_SC-70-6, F.Cu at (0.00, -25.8)
- added Q3: BC846BPN, Package_TO_SOT_SMD:SOT-363_SC-70-6, F.Cu at (0.00, -22.8)
- added Q4: BC846BS, Package_TO_SOT_SMD:SOT-363_SC-70-6, F.Cu at (2.75, -19.0)
- added Q5: BC846BS, Package_TO_SOT_SMD:SOT-363_SC-70-6, F.Cu at (-2.75, -19.0)
- added R100: 100R, Resistor_SMD:R_0402_1005Metric, F.Cu at (-31.2, 9.75)
- added R101: 100R, Resistor_SMD:R_0402_1005Metric, F.Cu at (-35.8, 17.2)
- added R102: 100R, Resistor_SMD:R_0402_1005Metric, F.Cu at (-34.2, 18.8)
- added R103: 100R, Resistor_SMD:R_0402_1005Metric, F.Cu at (-26.8, 15.2)
- added R104: 100R, Resistor_SMD:R_0402_1005Metric, F.Cu at (-26.8, 14.2)
- added R105: 100R, Resistor_SMD:R_0402_1005Metric, F.Cu at (-26.8, 13.2)
- added R106: 100R, Resistor_SMD:R_0402_1005Metric, F.Cu at (-26.8, 12.2)
- added R107: 100R, Resistor_SMD:R_0402_1005Metric, F.Cu at (-26.8, 11.2)
- added R109: 100R, Resistor_SMD:R_0402_1005Metric, F.Cu at (-34.2, 9.75)
- added R110: 100R, Resistor_SMD:R_0402_1005Metric, F.Cu at (-35.2, 9.75)
- added R111: 100R, Resistor_SMD:R_0402_1005Metric, F.Cu at (-35.8, 11.2)
- added R112: 100R, Resistor_SMD:R_0402_1005Metric, F.Cu at (-35.8, 12.2)
- added R113: 100R, Resistor_SMD:R_0402_1005Metric, F.Cu at (-35.8, 13.2)
- added R114: 100R, Resistor_SMD:R_0402_1005Metric, F.Cu at (-35.8, 14.2)
- added R115: 100R, Resistor_SMD:R_0402_1005Metric, F.Cu at (-35.8, 15.2)
- added R116: 100R, Resistor_SMD:R_0402_1005Metric, F.Cu at (-35.8, 16.2)
- added R119: 100R, Resistor_SMD:R_0402_1005Metric, F.Cu at (-26.8, 18.2)
- added R120: 100R, Resistor_SMD:R_0402_1005Metric, F.Cu at (-26.8, 17.2)
- added R121: 100R, Resistor_SMD:R_0402_1005Metric, F.Cu at (-26.8, 16.2)
- added R122: 100R, Resistor_SMD:R_0402_1005Metric, F.Cu at (-29.2, 9.75)
- added R123: 100R, Resistor_SMD:R_0402_1005Metric, F.Cu at (-30.2, 9.75)
- added R124: 2.2k, Resistor_SMD:R_0402_1005Metric, F.Cu at (-30.2, 7.75)
- added R125: 2.2k, Resistor_SMD:R_0402_1005Metric, F.Cu at (-29.2, 7.75)
- added R126: 10k, Resistor_SMD:R_0402_1005Metric, F.Cu at (-28.2, 9.75)
- added R200: NM, Resistor_SMD:R_0402_1005Metric, F.Cu at (43.0, 9.50)
- added R201: 3.3k, Resistor_SMD:R_0402_1005Metric, F.Cu at (43.0, 10.5)
- added R202: NM, Resistor_SMD:R_0402_1005Metric, F.Cu at (43.0, 8.50)
- added R203: 0R, Resistor_SMD:R_0402_1005Metric, F.Cu at (43.0, 7.50)
- added R204: 1M, Resistor_SMD:R_0402_1005Metric, F.Cu at (43.0, 13.5)
- added R205: 130k, Resistor_SMD:R_0402_1005Metric, F.Cu at (41.5, 6.00)
- added R206: 180k, Resistor_SMD:R_0402_1005Metric, F.Cu at (33.5, 5.00)
- added R207: 62k, Resistor_SMD:R_0402_1005Metric, F.Cu at (34.0, 6.50)
- added R208: 100R, Resistor_SMD:R_0402_1005Metric, F.Cu at (43.0, 15.5)
- added R209: 100R, Resistor_SMD:R_0402_1005Metric, F.Cu at (43.0, 14.5)
- added R23: 100R, Resistor_SMD:R_0402_1005Metric, F.Cu at (-22.8, 7.50)
- added R24: 4.32k, Resistor_SMD:R_0402_1005Metric, F.Cu at (-2.50, 11.0)
- added R300: NM, Resistor_SMD:R_0402_1005Metric, F.Cu at (43.0, -2.50)
- added R301: 3.3k, Resistor_SMD:R_0402_1005Metric, F.Cu at (43.0, -1.50)
- added R302: NM, Resistor_SMD:R_0402_1005Metric, F.Cu at (43.0, -3.50)
- added R303: 0R, Resistor_SMD:R_0402_1005Metric, F.Cu at (43.0, -4.50)
- added R304: 1M, Resistor_SMD:R_0402_1005Metric, F.Cu at (43.0, 1.50)
- added R305: 130k, Resistor_SMD:R_0402_1005Metric, F.Cu at (41.5, -6.00)
- added R306: 180k, Resistor_SMD:R_0402_1005Metric, F.Cu at (33.5, -7.00)
- added R307: 62k, Resistor_SMD:R_0402_1005Metric, F.Cu at (34.0, -5.50)
- added R308: 100R, Resistor_SMD:R_0402_1005Metric, F.Cu at (43.0, 3.50)
- added R309: 100R, Resistor_SMD:R_0402_1005Metric, F.Cu at (43.0, 2.50)
- added R33: 33R, Resistor_SMD:R_0402_1005Metric, F.Cu at (3.50, 6.25)
- added R4: 33k, Resistor_SMD:R_0402_1005Metric, F.Cu at (-2.75, -24.5)
- added R40: 100R, Resistor_SMD:R_0402_1005Metric, F.Cu at (11.0, 4.75)
- added R48: 100k, Resistor_SMD:R_0402_1005Metric, F.Cu at (10.8, 25.5)
- added R49: 33k, Resistor_SMD:R_0402_1005Metric, F.Cu at (0.00, -19.2)
- added R50: 33k, Resistor_SMD:R_0402_1005Metric, F.Cu at (-5.50, -19.0)
- added R51: 33k, Resistor_SMD:R_0402_1005Metric, F.Cu at (5.50, -19.0)
- added R52: 33k, Resistor_SMD:R_0402_1005Metric, F.Cu at (0.00, -20.2)
- added R53: 33k, Resistor_SMD:R_0402_1005Metric, F.Cu at (0.00, -18.2)
- added R54: 33k, Resistor_SMD:R_0402_1005Metric, F.Cu at (-5.50, -18.0)
- added R55: 2.2k, Resistor_SMD:R_0402_1005Metric, F.Cu at (-38.2, 6.00)
- added R57: 2.2k, Resistor_SMD:R_0402_1005Metric, F.Cu at (-38.2, 16.0)
- added R9: 33k, Resistor_SMD:R_0402_1005Metric, F.Cu at (-2.75, -26.5)
- added SW1: SW_Push, Button_Switch_SMD:SW_SPST_PTS810, F.Cu at (0.00, 25.2)
- added SW2: SW_Push, Button_Switch_SMD:SW_SPST_PTS810, F.Cu at (-41.8, 2.50)
- added SW3: SW_Push, Button_Switch_SMD:SW_SPST_PTS810, F.Cu at (-41.8, -2.50)
- added SW4: SW_Push, Button_Switch_SMD:SW_SPST_PTS810, F.Cu at (-41.8, 7.50)
- added SW5: SW_Push, Button_Switch_SMD:SW_SPST_PTS810, F.Cu at (-41.8, 12.5)
- added SW6: SW_Push, Button_Switch_SMD:SW_SPST_PTS810, F.Cu at (-41.8, 17.5)
- added U100: STM32F042G4Ux, Package_DFN_QFN:QFN-28_4x4mm_P0.5mm, F.Cu at (-31.2, 14.2)
- added U101: USBLC6-2SC6, Package_TO_SOT_SMD:SOT-23-6, F.Cu at (-29.8, 19.8)
- added U200: L6986, Package_SO:HTSSOP-16-1EP_4.4x5mm_P0.65mm_EP3x3mm, F.Cu at (37.0, 10.0)
- added U300: L6986, Package_SO:HTSSOP-16-1EP_4.4x5mm_P0.65mm_EP3x3mm, F.Cu at (37.0, -2.00)
- added U5: 74LS125, Package_SO:TSSOP-14_4.4x5mm_P0.65mm, F.Cu at (0.00, -14.8)
- C12, C6: value 100n -> 100p
- C20: renamed from C36; value 10n -> 100n
- C21: value 100n -> 4.7u
- C22: value 100p -> 100n
- C23: renamed from C39; value 10n -> 100n
- C26: renamed from C42; value 10n -> 100n
- C29: renamed from C45; value 10n -> 100n
- C33: value 100p -> 10n
- D1, D2: value LED_Small -> BAS516; footprint Diode_SMD:D_0603_1608Metric -> Diode_SMD:D_SOD-523
- J100: value Conn_01x02_Female -> JST_XH_S2B; footprint Connector_JST:JST_PH_B2B-PH-K_1x02_P2.00mm_Vertical -> Connector_JST:JST_XH_S2B-XH-A_1x02_P2.50mm_Horizontal
- JP1: value Jumper_NC_Dual -> Jumper_3_Bridged12
- PCB1: value Board_Module -> 90x55; footprint PCB_Board:90x55 -> Farving_Labs_Library:PCB_Board_90x55
- R17: value 0R -> 100R; footprint Diode_SMD:D_0402_1005Metric -> Resistor_SMD:R_0402_1005Metric
- R18: value 18k -> 100R; footprint Diode_SMD:D_0402_1005Metric -> Resistor_SMD:R_0402_1005Metric
- R19: value 300k -> 100R; footprint Diode_SMD:D_0402_1005Metric -> Resistor_SMD:R_0402_1005Metric
- R20: value 1M -> 100R; footprint Diode_SMD:D_0402_1005Metric -> Resistor_SMD:R_0402_1005Metric
- R21: value 33R -> 100R
- R22, R6: value 66R -> 33k
- R42: value 100R -> 10k
- R43, R44, R45: value 100R -> 33k
- R46: value 100R -> 100k
- R47: value 4.32k -> 2.2k
- R56: value 33R -> 2.2k
- U4: value LT8608 -> 74LS125; footprint Package_SO:MSOP-10-1EP_3x3mm_P0.5mm_EP1.68x1.88mm -> Package_SO:TSSOP-14_4.4x5mm_P0.65mm
- moved C12 57.9 mm to (-17.8, 7.50), turned to 90 degrees
- moved R21 56.6 mm to (-20.8, 7.50), turned to 90 degrees
- moved R20 54.1 mm to (-18.8, 7.50), turned to 90 degrees
- moved C6 52.3 mm to (-13.8, 7.50), turned to 90 degrees
- moved R19 52.0 mm to (-16.8, 7.50), turned to 90 degrees
- moved R18 51.3 mm to (-14.8, 7.50), turned to 90 degrees
- moved D1 51.1 mm to (5.75, -21.8), turned to 180 degrees
- moved R17 50.0 mm to (-12.8, 7.50), turned to 90 degrees
- moved D2 48.5 mm to (5.75, -20.2), turned to 180 degrees
- moved R42 44.0 mm to (2.75, -25.5), turned to 180 degrees
- moved R56 43.5 mm to (-38.2, 11.0), turned to 270 degrees
- moved R43 42.2 mm to (2.75, -24.5), turned to 0 degrees
- moved R44 40.6 mm to (2.75, -23.5), turned to 0 degrees
- moved R22 38.3 mm to (-2.75, -23.5), turned to 0 degrees
- moved R45 37.6 mm to (-2.75, -22.5), turned to 0 degrees
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- renumbered C17 to C1, C26 to C10, C27 to C11, C29 to C13, C30 to C14, C32 to C16, C34 to C18, C35 to C19, C18 to C2, C19 to C3, C48 to C32, C20 to C4, C23 to C7, C24 to C8, C25 to C9, R29 to R1, R34 to R10, R35 to R11, R36 to R12, R37 to R13, R38 to R14, R39 to R15, R40 to R16, R30 to R2, R48 to R25, R49 to R26, R50 to R27, R51 to R28, R52 to R29, R53 to R30, R54 to R31, R55 to R32, R57 to R34, R58 to R35, R59 to R36, R60 to R37, R61 to R38, R62 to R39, R31 to R5, R32 to R7, R33 to R8, U7 to U2, U8 to U3
Connections:
- net /MISO_M renamed /SDA_M
- net /MOSI_M renamed Net-(U2-Pad27)
- C10 pad 2: GND -> GNDS
- C11 pad 2: GND -> GNDS
- C12 pad 2: Net-(C12-Pad2) -> GND
- C14 pad 1: Net-(C30-Pad1) -> Net-(C14-Pad1)
- C21 pad 1: /DSP/AVDD -> Net-(C21-Pad1)
- C22 pad 1: Net-(C22-Pad1) -> /BTN_RESET
- C33 pad 1: Net-(C33-Pad1) -> /PUSH_BTN0
- C4 pad 1: Net-(C20-Pad1) -> Net-(C4-Pad1)
- C6 pad 2: Net-(C6-Pad2) -> GND
- C8 pad 1: Net-(C24-Pad1) -> Net-(C8-Pad1)
- C9 pad 1: Net-(C25-Pad1) -> Net-(C9-Pad1)
- D1 pad 1: Net-(D1-Pad1) -> /DSP_SHDN
- D1 pad 2: +5V -> Net-(D1-Pad2)
- D2 pad 1: Net-(D2-Pad1) -> /MCU_SHDN
- D2 pad 2: +5V -> Net-(D1-Pad2)
- J100 pad 1: VDD -> Net-(C100-Pad1)
- J101 pad 1: +3V3 -> /I2S_MCLKI0
- J101 pad 10: /COM_CSI0 -> GND
- J101 pad 11: Net-(J101-Pad11) -> /I2C_SCL
- J101 pad 12: Net-(J101-Pad12) -> GND
- J101 pad 13: Net-(J101-Pad13) -> /I2C_SDA
- J101 pad 15: Net-(J101-Pad15) -> /nSHDN
- J101 pad 17: Net-(J101-Pad17) -> /nMUTE
- J101 pad 19: /MCLK -> +3V3
- J101 pad 2: +5V -> GND
- J101 pad 20: GND -> +5V
- J101 pad 3: GND -> /I2S_BCLKI0
- J101 pad 5: /SHDN -> /I2S_LRCLKI0
- J101 pad 6: /MUTE -> GND
- J101 pad 7: /COM_CLK -> /I2S_SDI0
- J101 pad 8: /COM_SDAO -> GND
- J101 pad 9: /COM_SDAI -> Net-(J101-Pad9)
- J102 pad 1: +3V3 -> /I2S_MCLKO0
- J102 pad 10: /COM_CSO0 -> GND
- J102 pad 11: Net-(J102-Pad11) -> /I2C_SCL
- J102 pad 12: Net-(J102-Pad12) -> GND
- J102 pad 13: Net-(J102-Pad13) -> /I2C_SDA
- J102 pad 15: Net-(J102-Pad15) -> /nSHDN
- J102 pad 17: Net-(J102-Pad17) -> /nMUTE
- J102 pad 19: /MCLK -> +3V3
- J102 pad 2: +5V -> GND
- J102 pad 20: GND -> +5V
- J102 pad 3: GND -> /I2S_BCLKO0
- J102 pad 5: /SHDN -> /I2S_LRCLKO0
- J102 pad 6: /MUTE -> GND
- J102 pad 7: /COM_CLK -> /I2S_SDO0
- J102 pad 8: /COM_SDAO -> GND
- J102 pad 9: /COM_SDAI -> Net-(J102-Pad9)
- J103 pad 4: Net-(J103-Pad4) -> /USBi_DET
- J103 pad 6: /USB_Reset -> /USB_RESET
- JP1 pad 1: /SCLK_M -> GND
- JP1 pad 2: /COM_CLK -> /ADAU1452_SELFBOOT
- JP1 pad 3: /Ext_SCLK -> +3V3
- R1 pad 2: /DSP/BCLKI0 -> /I2S_BCLKI0
- R10 pad 2: /SDI1 -> /I2S_SDI1
- R13 pad 2: /SDI2 -> /DSP/SDI2
- R16 pad 2: /SDI3 -> /DSP/SDI3
- R17 pad 1: Net-(C10-Pad1) (its old number) -> Net-(C4-Pad1)
- R17 pad 2: Net-(R17-Pad2) -> /DSP/ADC0
- R18 pad 1: Net-(R18-Pad1) -> Net-(C6-Pad1)
- R18 pad 2: GND -> /DSP/ADC1
- R19 pad 1: Net-(C13-Pad2) -> Net-(C8-Pad1)
- R19 pad 2: GND -> /DSP/ADC2
- R2 pad 2: /DSP/LRCLKI0 -> /I2S_LRCLKI0
- R20 pad 1: +3V3 -> Net-(C12-Pad1)
- R20 pad 2: Net-(C13-Pad2) -> /DSP/ADC3
- R21 pad 1: Net-(J102-Pad15) -> Net-(C15-Pad1)
- R21 pad 2: /DSP/BCLKO3 -> /DSP/ADC4
- R22 pad 1: GND -> +3V3
- R22 pad 2: /MCLK -> Net-(Q2-Pad3)
- R27 pad 2: /DSP/LRCLKO2 -> /I2S_LRCLKO1
- R28 pad 2: /DSP/BCLKO2 -> /I2S_BCLKO1
- R29 pad 2: /DSP/SDO2 -> /I2S_SDO1
- R3 pad 1: Net-(J103-Pad4) -> /USBi_DET
- R30 pad 2: /DSP/LRCLKO3 -> /I2S_LRCLKO0
- R31 pad 2: /DSP/BCLKO3 -> /I2S_BCLKO0
- R32 pad 2: /DSP/SDO3 -> /I2S_SDO0
- R41 pad 1: Net-(C20-Pad1) -> /I2C_SCL
- R41 pad 2: /DSP/ADC0 -> /SCL_M
- R42 pad 1: Net-(C22-Pad1) -> +3V3
- R42 pad 2: /DSP/ADC1 -> Net-(Q2-Pad5)
- R43 pad 1: Net-(C24-Pad1) -> Net-(Q2-Pad5)
- R43 pad 2: /DSP/ADC2 -> GND
- R44 pad 1: Net-(C28-Pad1) -> Net-(Q3-Pad2)
- R44 pad 2: /DSP/ADC3 -> GND
- R45 pad 1: Net-(C31-Pad1) -> +3V3
- R45 pad 2: /DSP/ADC4 -> Net-(D4-Pad1)
- R46 pad 1: Net-(C33-Pad1) -> Net-(J110-Pad4)
- R46 pad 2: /DSP/ADC5 -> GND
- R47 pad 1: Net-(C30-Pad1) -> +3V3
- R47 pad 2: Net-(C25-Pad1) -> /PUSH_BTN0
- R5 pad 2: /SDI0 -> /I2S_SDI0
- R56 pad 1: Net-(R56-Pad1) -> +3V3
- R56 pad 2: /MCLK -> /PUSH_BTN2
- R6 pad 1: /MCLK -> +3V3
- R6 pad 2: GND -> Net-(Q2-Pad6)
- R7 pad 2: /DSP/BCLKI1 -> /I2S_BCLKI1
- R8 pad 2: /DSP/LRCLKI1 -> /I2S_LRCLKI1
- U2 pad 10: Net-(C24-Pad1) -> Net-(C8-Pad1)
- U2 pad 11: Net-(C28-Pad1) -> Net-(C12-Pad1)
- U2 pad 12: Net-(C31-Pad1) -> Net-(C15-Pad1)
- U2 pad 13: Net-(C33-Pad1) -> Net-(C17-Pad1)
- U2 pad 16: Net-(C30-Pad1) -> Net-(C14-Pad1)
- U2 pad 23: Net-(R56-Pad1) -> Net-(R33-Pad1)
- U2 pad 24: /DSP/nRESET -> /ADAU1452_nRESET
- U2 pad 28: /SCLK_M -> /SCL_M
- U2 pad 34: /DSP/SELFBOOT -> /ADAU1452_SELFBOOT
- U2 pad 45: /SHDN -> /DSP_MUTE
- U2 pad 46: /MUTE -> /DSP_SHDN
- U2 pad 8: Net-(C20-Pad1) -> Net-(C4-Pad1)
- U2 pad 9: Net-(C22-Pad1) -> Net-(C6-Pad1)
- U3 pad 3: VDD -> +3V3
- U3 pad 6: /SCLK_M -> /SCL_M
- U3 pad 7: VDD -> +3V3
- U3 pad 8: VDD -> +3V3
- U4 pad 1: Net-(C12-Pad1) -> /USBi_DET
- U4 pad 10: Net-(R16-Pad2) -> /USBi_DET
- U4 pad 11: GND -> /SCLK
- U4 pad 2: Net-(C12-Pad2) -> /SPI_NSS
- U4 pad 3: Net-(C10-Pad1) (its old number) -> /SS
- U4 pad 4: Net-(R18-Pad1) -> /USBi_DET
- U4 pad 5: Net-(R17-Pad2) -> /SPI1_MOSI
- U4 pad 6: Net-(C13-Pad2) -> /MOSI
- U4 pad 7: Net-(C11-Pad1) (its old number) -> GND
- U4 pad 8: /PG_3V3 -> /MISO
- U4 pad 9: +5V -> /SPI1_MISO
- Y1 pad 2: GND -> GNDS
- Y1 pad 4: GND -> GNDS
Routing:
- net /3V3_RESET: track 0.00 -> 134.4 mm, vias 0 -> 3
- net /I2C_SCL: track 0.00 -> 133.7 mm, vias 0 -> 1
- net /I2C_SDA: track 0.00 -> 133.7 mm, vias 0 -> 1
- net /MCU_SHDN: track 0.00 -> 89.1 mm
- net +3V3: track 19.4 -> 106.7 mm, vias 5 -> 39
- net /nMUTE: track 0.00 -> 85.7 mm, vias 0 -> 1
- net /nSHDN: track 0.00 -> 83.7 mm, vias 0 -> 1
- net /ADAU1452_SELFBOOT: track 0.00 -> 83.5 mm, vias 0 -> 2
- net /USBi_DET: track 0.00 -> 72.0 mm, vias 0 -> 4
- net /MCU_MUTE: track 0.00 -> 70.1 mm
- net /SCLK: track 0.00 -> 47.6 mm
- net /SS: track 0.00 -> 47.0 mm
- net /I2S_MCLKI0: track 0.00 -> 46.5 mm
- net /DSP/SPDIFIN: track 0.00 -> 46.0 mm, vias 0 -> 1
- net /SPI1_MOSI: track 0.00 -> 44.6 mm, vias 0 -> 2
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- added copper zone on F.Cu, net +3V3
- added copper zone on In2.Cu, net +3V3
- added copper zone on F.Cu, net +5V
- added copper zone on In2.Cu, net +5V
- added copper zone on F.Cu, net /DSP/DVDD
- added copper zone on In2.Cu, net /DSP/DVDD
- added copper zone on B.Cu, net GND
- added copper zone on F.Cu, net GND
- added copper zone on In1.Cu, net GND
- added copper zone on B.Cu, net GNDS
- added copper zone on F.Cu, net Net-(C100-Pad1)
- added copper zone on F.Cu, net Net-(L200-Pad1)
- added copper zone on F.Cu, net Net-(L300-Pad1)
- added copper zone on F.Cu, net VDD
Other:
- rule via_min_size: 0.4 -> 0.6
- board text added: "Farving Acoustics FA-Core 1x1 1000004-2.0.0"
