File: KiCad/Core 1x1/Core 1x1.sch (KiCad schematic (older format))
At the start: 102 parts, among them J100 Conn_01x02_Female, J101 02x10, J102 02x10, J103 Conn_02x05_Odd_Even, J12 Conn_01x09_Male, J13 Conn_01x03_Male, U3 LT8608, U4 LT8608

Commit message: Pre-release commit
Parts:
- removed C1, C14, C8, C9: 10u, Capacitor_SMD:C_0805_2012Metric, symbol Device:C_Small
- removed C10, C2: 1u, Capacitor_SMD:C_0402_1005Metric, symbol Device:C_Small
- removed C11, C3: 10n, Capacitor_SMD:C_0402_1005Metric, symbol Device:C_Small
- removed C12, C6: 100n, Capacitor_SMD:C_0402_1005Metric, symbol Device:C_Small
- removed C13, C7: 10p, Capacitor_SMD:C_0402_1005Metric, symbol Device:C_Small
- removed D1, D2: LED_Small, Diode_SMD:D_0603_1608Metric, symbol Device:LED_Small
- removed J12: Conn_01x09_Male, Connector_JST:JST_PH_B9B-PH-K_1x09_P2.00mm_Vertical, symbol Connector:Conn_01x09_Male
- removed J13: Conn_01x03_Male, Connector_JST:JST_PH_B3B-PH-K_1x03_P2.00mm_Vertical, symbol Connector:Conn_01x03_Male
- removed JP1, JP2, JP3: Jumper_NC_Dual, Connector_PinHeader_2.54mm:PinHeader_1x03_P2.54mm_Vertical, symbol Device:Jumper_NC_Dual
- removed L1, L2: 10u, Inductor_SMD:L_Bourns_SRP7028A_7.3x6.6mm, symbol Device:L_Small
- removed R1, R2, R21, R25, R26, R5: 33R, Resistor_SMD:R_0402_1005Metric, symbol Device:R_Small
- removed R11, R18: 18k, Diode_SMD:D_0402_1005Metric, symbol Device:R_Small
- removed R12: 180k, Diode_SMD:D_0402_1005Metric, symbol Device:R_Small
- removed R13, R20: 1M, Diode_SMD:D_0402_1005Metric, symbol Device:R_Small
- removed R14, R15: 100R, Diode_SMD:D_0402_1005Metric, symbol Device:R_Small
- removed R16, R17, R7, R8: 0R, Diode_SMD:D_0402_1005Metric, symbol Device:R_Small
- removed R19: 300k, Diode_SMD:D_0402_1005Metric, symbol Device:R_Small
- removed R?: 1k, Resistor_SMD:R_0402_1005Metric, symbol Device:R_Small
- removed R?: 100k, Resistor_SMD:R_0402_1005Metric, symbol Device:R_Small
- removed SW?: SW_Push, symbol Switch:SW_Push
- removed TP1, TP10, TP11, TP12, TP13, TP14, TP15, TP16, TP17, TP18, TP19, TP2, TP20, TP21, TP22, TP23, TP24, TP3, TP31, TP32, TP33, TP34, TP35, TP36, TP37, TP38, TP39, TP4, TP40, TP41, TP42, TP43, TP44, TP45, TP46, TP47, TP48, TP5, TP6, TP7, TP8, TP9: TestPoint, TestPoint:TestPoint_Pad_D1.0mm, symbol Connector:TestPoint
- removed U3, U4: LT8608, Package_SO:MSOP-10-1EP_3x3mm_P0.5mm_EP1.68x1.88mm, symbol Core-1x1-rescue:LT8606-FA-Library-Core-2x2-rescue
- removed U?: STM811, Package_TO_SOT_SMD:SOT-143, symbol Power_Supervisor:MAX811LEUS-T
- added C100, C101: 4.7u, Capacitor_SMD:C_0805_2012Metric, symbol Device:C_Small
- added C102, C21: 4.7u, Capacitor_SMD:C_0402_1005Metric, symbol Device:C_Small
- added C103, C22, C34, C35: 100n, Capacitor_SMD:C_0402_1005Metric, symbol Device:C_Small
- added C106, C24, C25, C27, C33: 10n, Capacitor_SMD:C_0402_1005Metric, symbol Device:C_Small
- added C107: 1u, Capacitor_SMD:C_0402_1005Metric, symbol Device:C_Small
- added D1, D10, D11, D2, D4, D5, D6, D7, D8, D9: BAS516, Diode_SMD:D_SOD-523, symbol Device:D_Small
- added J1: TC2030, Connector:Tag-Connect_TC2030-IDC-NL_2x03_P1.27mm_Vertical, symbol Connector_Generic:Conn_02x03_Odd_Even
- added J104, J109: 02x10, Connector_PinHeader_2.54mm:PinHeader_2x10_P2.54mm_Vertical, symbol Connector_Generic:Conn_02x10_Odd_Even
- added J105, J106, J107, J108: Conn_02x03_Odd_Even, Connector_PinHeader_2.54mm:PinHeader_2x03_P2.54mm_Vertical, symbol Connector_Generic:Conn_02x03_Odd_Even
- added J110: USB_OTG, Connector_USB:USB_Micro-B_Molex-105017-0001, symbol Connector:USB_OTG
- added J2, J3: JST_XH_B2B, Connector_JST:JST_XH_B2B-XH-A_1x02_P2.50mm_Vertical, symbol Connector:Conn_01x02_Male
- added JP1: Jumper_3_Bridged12, Connector_PinHeader_2.54mm:PinHeader_1x03_P2.54mm_Vertical, symbol Jumper:Jumper_3_Bridged12
- added L100: 4.7u, Farving_Labs_Library:L_Pulse_PA4546.XXXNLT, symbol Device:L_Small
- added Q2, Q4, Q5: BC846BS, Package_TO_SOT_SMD:SOT-363_SC-70-6, symbol Device:Q_DUAL_NPN_NPN_E1B1C2E2B2C1
- added Q3: BC846BPN, Package_TO_SOT_SMD:SOT-363_SC-70-6, symbol Device:Q_DUAL_NPN_PNP_E1B1C2E2B2C1
- added R100, R101, R102, R103, R104, R105, R106, R107, R109, R110, R111, R112, R113, R114, R115, R116, R119, R120, R121, R122, R123, R40, R41: 100R, Resistor_SMD:R_0402_1005Metric, symbol Device:R_Small
- added R124, R125, R47, R55, R56, R57: 2.2k, Resistor_SMD:R_0402_1005Metric, symbol Device:R_Small
- added R126, R42: 10k, Resistor_SMD:R_0402_1005Metric, symbol Device:R_Small
- added R4, R43, R44, R45, R49, R50, R51, R52, R53, R54, R9: 33k, Resistor_SMD:R_0402_1005Metric, symbol Device:R_Small
- added R46, R48: 100k, Resistor_SMD:R_0402_1005Metric, symbol Device:R_Small
- added SW1, SW2, SW3, SW4, SW5, SW6: SW_Push, Button_Switch_SMD:SW_SPST_PTS810, symbol Switch:SW_Push
- added U100: STM32F042G4Ux, Package_DFN_QFN:QFN-28_4x4mm_P0.5mm, symbol MCU_ST_STM32F0:STM32F042G4Ux
- added U101: USBLC6-2SC6, Package_TO_SOT_SMD:SOT-23-6, symbol Power_Protection:USBLC6-2SC6
- added U4, U5: 74LS125, Package_SO:TSSOP-14_4.4x5mm_P0.65mm, symbol 74xx:74LS125
- J100: value Conn_01x02_Female -> JST_XH_S2B; footprint Connector_JST:JST_PH_B2B-PH-K_1x02_P2.00mm_Vertical -> Connector_JST:JST_XH_S2B-XH-A_1x02_P2.50mm_Horizontal
- PCB1: value Board_Module -> 90x55; footprint PCB_Board:90x55 -> Farving_Labs_Library:PCB_Board_90x55; symbol Library:Board_Module -> Core-1x1-rescue:Board_Module-Library
- R22, R6: value 66R -> 33k
Connections:
- net labels added: 3V3_RESET, ADAU1452_SELFBOOT, ADAU1452_nRESET, BOOT0, BTN_RESET, DSP_MUTE, DSP_SHDN, I2S_BCLKI0, I2S_BCLKI1, I2S_BCLKO0, I2S_BCLKO1, I2S_LRCLKI0, I2S_LRCLKI1, I2S_LRCLKO0, I2S_LRCLKO1, I2S_MCLK, I2S_MCLKI0, I2S_MCLKI1, I2S_MCLKO0, I2S_MCLKO1, I2S_SDI0, I2S_SDI1, I2S_SDO0, I2S_SDO1, MCU_DSP_RESET, MCU_MUTE, MCU_SHDN, MCU_nRST, PUSH_BTN0, PUSH_BTN1, PUSH_BTN2, PUSH_BTN3, SCL_M, SDA_M, SPI1_CLK, SPI1_MISO, SPI1_MOSI, SPI_NSS, SWCLK, SWDIO, SYNC, USB_D+, USB_D-, USB_DM, USB_DP, USB_RESET, USBi_DET, VBUS, nMUTE, nSHDN
- net labels removed: COM_CLK, COM_CSI0, COM_CSO0, COM_SDAI, COM_SDAO, Ext_SCLK, Ext_SDAI, Ext_SDAO, MCLK, MISO_M, MOSI_M, MUTE, PG_3V3, PG_5V, SCLK_M, SDI0, SDI1, SDI2, SDI3, SHDN, SPI_MISO, SPI_MOSI, SPI_SCK, SPI_SS0, SPI_SS1, SPI_SS2, SPI_SS3, SPI_SS4, USB_Reset
- wire segments 341 -> 567
Other:
- note added: "RESERVED"
- note added: "We are only using I2C to daughterboards for simplicity\nAll SPI only slaves must use a I2C-to-SPI-bridge"
- note removed: "ADAU1452<=500mA on 3V3\n100mA for each supply on each daughterboard\n5V <= 500mA\n3V3 <= 500mA + 500mA <= 1A \n2x LT8608 = 2x 1.5A"
- note removed: "Add Reset supervisor\nAdd reset button"
- note removed: "Add jumper for slave control IO"
- note removed: "SDA\nBCLK\nLRCLK\nMCLK"
- moved on the sheet: D3, J100, PCB1, R3
